File: PCB/ECEN 2440 Final Project/Radio Board.brd (EAGLE design)
At the start: 58.4 x 38.1 mm, 27 parts

Commit message: really important commit
Parts:
- added U$2: WOBBUFFET, Custom Library:WOBBUFFET
Other:
- board text added: "DRA818v Breakout Board"
- board text added: "T E A M R O C K E T ecen 2440 fall 2019 final project XuTao Ho | Dustin Horn | Giselle Koo"
Changed lines of the file:
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@@
 <setting verticaltext="up"/>
 </settings>
-<grid distance="0.05" unitdist="inch" unit="mm" style="lines" multiple="1" display="yes" altdistance="5" altunitdist="mil" altunit="inch"/>
+<grid distance="0.003333" unitdist="inch" unit="inch" style="lines" multiple="1" display="yes" altdistance="5" altunitdist="mil" altunit="inch"/>
 <layers>
 <layer number="1" name="Top" color="4" fill="1" visible="yes" active="yes"/>
@@
 <layer number="14" name="Route14" color="1" fill="6" visible="no" active="no"/>
 <layer number="15" name="Route15" color="4" fill="6" visible="no" active="no"/>
-<layer number="16" name="Bottom" color="1" fill="1" visible="yes" active="yes"/>
+<layer number="16" name="Bottom" color="1" fill="1" visible="no" active="yes"/>
 <layer number="17" name="Pads" color="2" fill="1" visible="yes" active="yes"/>
 <layer number="18" name="Vias" color="2" fill="1" visible="yes" active="yes"/>
@@
 <layer number="20" name="Dimension" color="24" fill="1" visible="yes" active="yes"/>
 <layer number="21" name="tPlace" color="7" fill="1" visible="yes" active="yes"/>
-<layer number="22" name="bPlace" color="7" fill="1" visible="yes" active="yes"/>
+<layer number="22" name="bPlace" color="7" fill="1" visible="no" active="yes"/>
 <layer number="23" name="tOrigins" color="15" fill="1" visible="yes" active="yes"/>
-<layer number="24" name="bOrigins" color="15" fill="1" visible="yes" active="yes"/>
+<layer number="24" name="bOrigins" color="15" fill="1" visible="no" active="yes"/>
 <layer number="25" name="tNames" color="7" fill="1" visible="yes" active="yes"/>
-<layer number="26" name="bNames" color="7" fill="1" visible="yes" active="yes"/>
+<layer number="26" name="bNames" color="7" fill="1" visible="no" active="yes"/>
 <layer number="27" name="tValues" color="7" fill="1" visible="no" active="yes"/>
 <layer number="28" name="bValues" color="7" fill="1" visible="no" active="yes"/>
@@
 <layer number="38" name="bTest" color="7" fill="1" visible="no" active="yes"/>
 <layer number="39" name="tKeepout" color="4" fill="11" visible="yes" active="yes"/>
-<layer number="40" name="bKeepout" color="1" fill="11" visible="yes" active="yes"/>
+<layer number="40" name="bKeepout" color="1" fill="11" visible="no" active="yes"/>
 <layer number="41" name="tRestrict" color="4" fill="10" visible="yes" active="yes"/>
-<layer number="42" name="bRestrict" color="1" fill="10" visible="yes" active="yes"/>
+<layer number="42" name="bRestrict" color="1" fill="10" visible="no" active="yes"/>
 <layer number="43" name="vRestrict" color="2" fill="10" visible="no" active="yes"/>
 <layer number="44" name="Drills" color="7" fill="1" visible="no" active="yes"/>
@@
 <layer number="50" name="dxf" color="7" fill="1" visible="no" active="no"/>
 <layer number="51" name="tDocu" color="7" fill="1" visible="yes" active="yes"/>
-<layer number="52" name="bDocu" color="7" fill="1" visible="yes" active="yes"/>
+<layer number="52" name="bDocu" color="7" fill="1" visible="no" active="yes"/>
 <layer number="53" name="tGND_GNDA" color="7" fill="9" visible="no" active="no"/>
 <layer number="54" name="bGND_GNDA" color="1" fill="9" visible="no" active="no"/>
@@
 <text x="27.686" y="0.254" size="1.27" layer="21">h/l</text>
 <text x="3.81" y="32.9946" size="1.778" layer="21" rot="R270">+</text>
+<text x="10.158984375" y="4.994834375" size="1.524" layer="21" font="vector" align="bottom-center">DRA818v
+Breakout Board</text>
+<text x="18.878778125" y="8.550478125" size="1.524" layer="22" font="vector" rot="SMR0" align="bottom-center">T E A M   R O C K E T
+ecen 2440 fall 2019
+final project
+XuTao Ho | Dustin Horn | Giselle Koo</text>
 </plain>
 <attributes>
@@
 </element>
 <element name="R6" library="rcl" library_urn="urn:adsk.eagle:library:334" package="R0805" package3d_urn="urn:adsk.eagle:package:23553/2" value="0R" x="16.256" y="35.433" smashed="yes" rot="R180">
-<attribute name="NAME" x="16.891" y="34.163" size="1.27" layer="25" rot="R180"/>
+<attribute name="NAME" x="18.4944" y="36.531703125" size="1.27" layer="25" rot="R270"/>
 <attribute name="POPULARITY" value="85" x="16.256" y="35.433" size="1.778" layer="27" rot="R180" display="off"/>
 <attribute name="SPICEPREFIX" value="R" x="16.256" y="35.433" size="1.778" layer="27" rot="R180" display="off"/>
@@
 </element>
 <element name="C5" library="rcl" library_urn="urn:adsk.eagle:library:334" package="PANASONIC_A" package3d_urn="urn:adsk.eagle:package:23418/2" value="" x="12.7" y="16.51" smashed="yes" rot="R270">
-<attribute name="NAME" x="14.45" y="18.16" size="1.016" layer="25" rot="R270"/>
+<attribute name="NAME" x="11.8936625" y="19.106203125" size="1.016" layer="25"/>
 <attribute name="POPULARITY" value="1" x="12.7" y="16.51" size="1.778" layer="27" rot="R270" display="off"/>
 <attribute name="SPICEPREFIX" value="C" x="12.7" y="16.51" size="1.778" layer="27" rot="R270" display="off"/>
@@
 </element>
 <element name="C6" library="rcl" library_urn="urn:adsk.eagle:library:334" package="PANASONIC_A" package3d_urn="urn:adsk.eagle:package:23418/2" value="" x="8.89" y="16.51" smashed="yes" rot="R270">
-<attribute name="NAME" x="10.64" y="18.16" size="1.016" layer="25" rot="R270"/>
+<attribute name="NAME" x="8.084040625" y="19.105821875" size="1.016" layer="25"/>
 <attribute name="POPULARITY" value="1" x="8.89" y="16.51" size="1.778" layer="27" rot="R270" display="off"/>
 <attribute name="SPICEPREFIX" value="C" x="8.89" y="16.51" size="1.778" layer="27" rot="R270" display="off"/>
@@
 <attribute name="VALUE" x="18.923" y="9.652" size="1.27" layer="27" rot="R90"/>
 </element>
+<element name="U$2" library="Custom Library" package="WOBBUFFET" value="WOBBUFFET" x="49.440390625" y="5.0794875" smashed="yes" rot="MR0"/>
 </elements>
 <signals>
@@
 <via x="16.891" y="15.875" extent="1-16" drill="0.35"/>
 <via x="5.969" y="15.24" extent="1-16" drill="0.35"/>
-<via x="9.525" y="5.715" extent="1-16" drill="0.35"/>
+<via x="9.44034375" y="2.667303125" extent="1-16" drill="0.35"/>
 <via x="24.13" y="16.002" extent="1-16" drill="0.35"/>
 <via x="26.797" y="18.542" extent="1-16" drill="0.35"/>
@@
 <via x="30.607" y="13.462" extent="1-16" drill="0.35"/>
 <via x="33.147" y="33.782" extent="1-16" drill="0.35"/>
-<via x="52.197" y="19.812" extent="1-16" drill="0.35"/>
-<via x="56.007" y="14.732" extent="1-16" drill="0.35"/>
-<via x="53.467" y="8.382" extent="1-16" drill="0.35"/>
+<via x="48.7260125" y="29.29371875" extent="1-16" drill="0.35"/>
+<via x="56.17631875" y="17.356403125" extent="1-16" drill="0.35"/>
+<via x="51.7738375" y="2.7099" extent="1-16" drill="0.35"/>
 </signal>
 <signal name="N$2">
@@
 </drawing>
 <compatibility>
+<note version="6.3" minversion="6.2.2" severity="warning">
+Since Version 6.2.2 text objects can contain more than one line,
+which will not be processed correctly with this version.
+</note>
 <note version="8.2" severity="warning">
 Since Version 8.2, EAGLE supports online libraries. The ids

Commit message: final board stuff
Parts:
- C4: value 500n -> 100n
- C5, C6: value (none) -> 2.2u
- CIN: value 100nF -> 10u
- COUT: value 1uF -> 10u
- R8, R9: value (none) -> 2R
Changed lines of the file:
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@@
 <attribute name="VALUE" x="52.705" y="30.099" size="1.27" layer="27" rot="R90"/>
 </element>
-<element name="CIN" library="rcl" library_urn="urn:adsk.eagle:library:334" package="PANASONIC_A" package3d_urn="urn:adsk.eagle:package:23418/2" value="100nF" x="6.477" y="35.179" smashed="yes" rot="R270">
+<element name="CIN" library="rcl" library_urn="urn:adsk.eagle:library:334" package="PANASONIC_A" package3d_urn="urn:adsk.eagle:package:23418/2" value="10u" x="6.477" y="35.179" smashed="yes" rot="R270">
 <attribute name="NAME" x="8.227" y="36.829" size="1.016" layer="25" rot="R270"/>
 <attribute name="POPULARITY" value="1" x="6.477" y="35.179" size="1.778" layer="27" rot="R270" display="off"/>
@@
 <attribute name="VALUE" x="3.652" y="36.829" size="1.016" layer="27" rot="R270"/>
 </element>
-<element name="COUT" library="rcl" library_urn="urn:adsk.eagle:library:334" package="PANASONIC_A" package3d_urn="urn:adsk.eagle:package:23418/2" value="1uF" x="3.556" y="17.653" smashed="yes" rot="R180">
+<element name="COUT" library="rcl" library_urn="urn:adsk.eagle:library:334" package="PANASONIC_A" package3d_urn="urn:adsk.eagle:package:23418/2" value="10u" x="3.556" y="17.653" smashed="yes" rot="R180">
 <attribute name="NAME" x="5.206" y="15.903" size="1.016" layer="25" rot="R180"/>
 <attribute name="POPULARITY" value="1" x="3.556" y="17.653" size="1.778" layer="27" rot="R180" display="off"/>
@@
 <attribute name="VALUE" x="-0.635" y="13.335" size="1.27" layer="27" rot="R270"/>
 </element>
-<element name="R8" library="rcl" library_urn="urn:adsk.eagle:library:334" package="R0805" package3d_urn="urn:adsk.eagle:package:23553/2" value="" x="12.573" y="10.922" smashed="yes" rot="R90">
+<element name="R8" library="rcl" library_urn="urn:adsk.eagle:library:334" package="R0805" package3d_urn="urn:adsk.eagle:package:23553/2" value="2R" x="12.573" y="10.922" smashed="yes" rot="R90">
 <attribute name="NAME" x="11.303" y="10.287" size="1.27" layer="25" rot="R90"/>
 <attribute name="POPULARITY" value="85" x="12.573" y="10.922" size="1.778" layer="27" rot="R90" display="off"/>
@@
 <attribute name="VALUE" x="15.113" y="10.287" size="1.27" layer="27" rot="R90"/>
 </element>
-<element name="R9" library="rcl" library_urn="urn:adsk.eagle:library:334" package="R0805" package3d_urn="urn:adsk.eagle:package:23553/2" value="" x="8.763" y="10.922" smashed="yes" rot="R90">
+<element name="R9" library="rcl" library_urn="urn:adsk.eagle:library:334" package="R0805" package3d_urn="urn:adsk.eagle:package:23553/2" value="2R" x="8.763" y="10.922" smashed="yes" rot="R90">
 <attribute name="NAME" x="7.493" y="10.287" size="1.27" layer="25" rot="R90"/>
 <attribute name="POPULARITY" value="85" x="8.763" y="10.922" size="1.778" layer="27" rot="R90" display="off"/>
@@
 <attribute name="VALUE" x="11.303" y="10.287" size="1.27" layer="27" rot="R90"/>
 </element>
-<element name="C5" library="rcl" library_urn="urn:adsk.eagle:library:334" package="PANASONIC_A" package3d_urn="urn:adsk.eagle:package:23418/2" value="" x="12.7" y="16.51" smashed="yes" rot="R270">
+<element name="C5" library="rcl" library_urn="urn:adsk.eagle:library:334" package="PANASONIC_A" package3d_urn="urn:adsk.eagle:package:23418/2" value="2.2u" x="12.7" y="16.51" smashed="yes" rot="R270">
 <attribute name="NAME" x="11.8936625" y="19.106203125" size="1.016" layer="25"/>
 <attribute name="POPULARITY" value="1" x="12.7" y="16.51" size="1.778" layer="27" rot="R270" display="off"/>
@@
 <attribute name="VALUE" x="9.875" y="18.16" size="1.016" layer="27" rot="R270"/>
 </element>
-<element name="C6" library="rcl" library_urn="urn:adsk.eagle:library:334" package="PANASONIC_A" package3d_urn="urn:adsk.eagle:package:23418/2" value="" x="8.89" y="16.51" smashed="yes" rot="R270">
+<element name="C6" library="rcl" library_urn="urn:adsk.eagle:library:334" package="PANASONIC_A" package3d_urn="urn:adsk.eagle:package:23418/2" value="2.2u" x="8.89" y="16.51" smashed="yes" rot="R270">
 <attribute name="NAME" x="8.084040625" y="19.105821875" size="1.016" layer="25"/>
 <attribute name="POPULARITY" value="1" x="8.89" y="16.51" size="1.778" layer="27" rot="R270" display="off"/>
@@
 <attribute name="VALUE" x="6.065" y="18.16" size="1.016" layer="27" rot="R270"/>
 </element>
-<element name="C4" library="rcl" library_urn="urn:adsk.eagle:library:334" package="C0805" package3d_urn="urn:adsk.eagle:package:23617/2" value="500n" x="16.383" y="10.922" smashed="yes" rot="R90">
+<element name="C4" library="rcl" library_urn="urn:adsk.eagle:library:334" package="C0805" package3d_urn="urn:adsk.eagle:package:23617/2" value="100n" x="16.383" y="10.922" smashed="yes" rot="R90">
 <attribute name="NAME" x="15.113" y="9.652" size="1.27" layer="25" rot="R90"/>
 <attribute name="POPULARITY" value="63" x="16.383" y="10.922" size="1.778" layer="27" rot="R90" display="off"/>
