File: PCB/ECEN 2440 Final Project/Custom Sheild-PCB.sch (EAGLE design)
At the start: 10 parts

Commit message: Work
Parts:
- added BATTERY: (no value), pinhead:PINHD-1X2
- added U$5: TEENSY_3.5/3.6_BASIC, Teensy356:TEENSY_3.5/3.6_BASIC
- added U$6: LFCN-160+, Custom Library:LFCN-160+
- added X1: (no value), adafruit:SMACONNECTOR_EDGE
Connections:
- new net +3V3: U$1.VDD, U$2.3V3, U$3.31, U$4.VBATT, U$5.3V3
- new net CD1: U$1.CARD_DETECT, U$3.48
- new net N$6: U$6.RF-OUT, X1.ANT
- new net VCC: BATTERY.2
- new net VSS: BATTERY.1
- net GND: now also U$1.VSS, U$5.GND, X1.GND1, X1.GND2, X1.GND3, X1.GND4
- net N$1: now also U$4.ANTENNA, U$6.RF-IN; no longer U$3.31
- net N$3: now also U$1.CARD_DETECT1; no longer U$4.VBATT
- net TEENSY_RX: now also U$5.0/RX
- net TEENSY_TX: now also U$5.1/TX
Changed lines of the file:
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@@
 <part name="GND7" library="supply1" library_urn="urn:adsk.eagle:library:371" deviceset="GND" device=""/>
 <part name="GND8" library="supply1" library_urn="urn:adsk.eagle:library:371" deviceset="GND" device=""/>
+<part name="U$5" library="Teensy356" deviceset="TEENSY_3.5/3.6_BASIC" device=""/>
+<part name="+3V1" library="supply1" library_urn="urn:adsk.eagle:library:371" deviceset="+3V3" device=""/>
+<part name="+3V2" library="supply1" library_urn="urn:adsk.eagle:library:371" deviceset="+3V3" device=""/>
+<part name="+3V3" library="supply1" library_urn="urn:adsk.eagle:library:371" deviceset="+3V3" device=""/>
+<part name="+3V4" library="supply1" library_urn="urn:adsk.eagle:library:371" deviceset="+3V3" device=""/>
+<part name="+3V5" library="supply1" library_urn="urn:adsk.eagle:library:371" deviceset="+3V3" device=""/>
+<part name="GND9" library="supply1" library_urn="urn:adsk.eagle:library:371" deviceset="GND" device=""/>
+<part name="U$6" library="Custom Library" deviceset="LFCN-160+" device=""/>
+<part name="X1" library="adafruit" library_urn="urn:adsk.eagle:library:420" deviceset="SMACONNECTOR" device="_EDGE" package3d_urn="urn:adsk.eagle:package:6240945/1"/>
+<part name="GND10" library="supply1" library_urn="urn:adsk.eagle:library:371" deviceset="GND" device=""/>
+<part name="GND11" library="supply1" library_urn="urn:adsk.eagle:library:371" deviceset="GND" device=""/>
+<part name="GND12" library="supply1" library_urn="urn:adsk.eagle:library:371" deviceset="GND" device=""/>
+<part name="GND13" library="supply1" library_urn="urn:adsk.eagle:library:371" deviceset="GND" device=""/>
+<part name="BATTERY" library="pinhead" library_urn="urn:adsk.eagle:library:325" deviceset="PINHD-1X2" device="" package3d_urn="urn:adsk.eagle:package:22435/2"/>
+<part name="P+1" library="supply1" library_urn="urn:adsk.eagle:library:371" deviceset="VCC" device=""/>
+<part name="VSS1" library="supply1" library_urn="urn:adsk.eagle:library:371" deviceset="VSS" device=""/>
 </parts>
 <sheets>
@@
 <attribute name="VALUE" x="160.02" y="-20.32" size="1.778" layer="96"/>
 </instance>
+<instance part="U$5" gate="G$1" x="88.9" y="-58.42" smashed="yes"/>
+<instance part="+3V1" gate="G$1" x="96.52" y="50.8" smashed="yes" rot="R270">
+<attribute name="VALUE" x="91.44" y="53.34" size="1.778" layer="96"/>
+</instance>
+<instance part="+3V2" gate="G$1" x="20.32" y="101.6" smashed="yes">
+<attribute name="VALUE" x="17.78" y="96.52" size="1.778" layer="96" rot="R90"/>
+</instance>
+<instance part="+3V3" gate="G$1" x="78.74" y="83.82" smashed="yes" rot="R90">
+<attribute name="VALUE" x="83.82" y="81.28" size="1.778" layer="96" rot="R180"/>
+</instance>
+<instance part="+3V4" gate="G$1" x="132.08" y="50.8" smashed="yes">
+<attribute name="VALUE" x="129.54" y="45.72" size="1.778" layer="96" rot="R90"/>
+</instance>
+<instance part="+3V5" gate="G$1" x="66.04" y="-81.28" smashed="yes" rot="R90">
+<attribute name="VALUE" x="71.12" y="-83.82" size="1.778" layer="96" rot="R180"/>
+</instance>
+<instance part="GND9" gate="1" x="66.04" y="-45.72" smashed="yes" rot="R270">
+<attribute name="VALUE" x="63.5" y="-43.18" size="1.778" layer="96" rot="R270"/>
+</instance>
+<instance part="U$6" gate="G$1" x="187.96" y="25.4" smashed="yes"/>
+<instance part="X1" gate="G$1" x="223.52" y="27.94" smashed="yes">
+<attribute name="NAME" x="233.68" y="30.48" size="1.27" layer="95"/>
+<attribute name="VALUE" x="231.14" y="27.94" size="1.27" layer="95"/>
+</instance>
+<instance part="GND10" gate="1" x="220.98" y="17.78" smashed="yes">
+<attribute name="VALUE" x="218.44" y="15.24" size="1.778" layer="96"/>
+</instance>
+<instance part="GND11" gate="1" x="226.06" y="17.78" smashed="yes">
+<attribute name="VALUE" x="223.52" y="15.24" size="1.778" layer="96"/>
+</instance>
+<instance part="GND12" gate="1" x="220.98" y="38.1" smashed="yes" rot="R180">
+<attribute name="VALUE" x="223.52" y="40.64" size="1.778" layer="96" rot="R180"/>
+</instance>
+<instance part="GND13" gate="1" x="226.06" y="38.1" smashed="yes" rot="R180">
+<attribute name="VALUE" x="228.6" y="40.64" size="1.778" layer="96" rot="R180"/>
+</instance>
+<instance part="BATTERY" gate="G$1" x="-38.1" y="45.72" smashed="yes" rot="R180">
+<attribute name="NAME" x="-31.75" y="40.005" size="1.778" layer="95" rot="R180"/>
+<attribute name="VALUE" x="-31.75" y="50.8" size="1.778" layer="96" rot="R180"/>
+</instance>
+<instance part="P+1" gate="VCC" x="-25.4" y="48.26" smashed="yes">
+<attribute name="VALUE" x="-27.94" y="45.72" size="1.778" layer="96" rot="R90"/>
+</instance>
+<instance part="VSS1" gate="G$1" x="-25.4" y="40.64" smashed="yes">
+<attribute name="VALUE" x="-27.94" y="35.56" size="1.778" layer="96" rot="R90"/>
+</instance>
 </instances>
 <busses>
@@
 <wire x1="-2.54" y1="35.56" x2="2.54" y2="35.56" width="0.1524" layer="91"/>
 <label x="-2.54" y="35.56" size="1.27" layer="95" rot="R180" xref="yes"/>
-</segment>
-</net>
-<net name="N$3" class="0">
-<segment>
-<pinref part="U$4" gate="G$1" pin="VBATT"/>
-<wire x1="132.08" y1="48.26" x2="132.08" y2="45.72" width="0.1524" layer="91"/>
 </segment>
 </net>
@@
 <wire x1="76.2" y1="76.2" x2="81.28" y2="76.2" width="0.1524" layer="91"/>
 <junction x="81.28" y="76.2"/>
+<pinref part="U$1" gate="G$1" pin="VSS"/>
+<wire x1="81.28" y1="81.28" x2="81.28" y2="76.2" width="0.1524" layer="91"/>
 </segment>
 <segment>
@@
 <pinref part="GND8" gate="1" pin="GND"/>
 </segment>
-</net>
-<net name="N$1" class="0">
-<segment>
-<pinref part="U$3" gate="MSP432" pin="31"/>
-<wire x1="93.98" y1="50.8" x2="86.36" y2="50.8" width="0.1524" layer="91"/>
+<segment>
+<pinref part="U$5" gate="G$1" pin="GND"/>
+<pinref part="GND9" gate="1" pin="GND"/>
+</segment>
+<segment>
+<pinref part="X1" gate="G$1" pin="GND3"/>
+<pinref part="GND10" gate="1" pin="GND"/>
+</segment>
+<segment>
+<pinref part="X1" gate="G$1" pin="GND4"/>
+<pinref part="GND11" gate="1" pin="GND"/>
+</segment>
+<segment>
+<pinref part="X1" gate="G$1" pin="GND1"/>
+<pinref part="GND12" gate="1" pin="GND"/>
+</segment>
+<segment>
+<pinref part="X1" gate="G$1" pin="GND2"/>
+<pinref part="GND13" gate="1" pin="GND"/>
 </segment>
 </net>
@@
 <label x="48.26" y="2.54" size="1.27" layer="95" rot="R90" xref="yes"/>
 </segment>
+<segment>
+<pinref part="U$5" gate="G$1" pin="1/TX"/>
+<wire x1="68.58" y1="-50.8" x2="66.04" y2="-50.8" width="0.1524" layer="91"/>
+<label x="66.04" y="-50.8" size="1.27" layer="95" rot="R180" xref="yes"/>
+</segment>
 </net>
 <net name="TEENSY_RX" class="0">
@@
 <label x="45.72" y="-27.94" size="1.27" layer="95" rot="R270" xref="yes"/>
 <wire x1="45.72" y1="-10.16" x2="45.72" y2="-27.94" width="0.1524" layer="91"/>
+</segment>
+<segment>
+<pinref part="U$5" gate="G$1" pin="0/RX"/>
+<wire x1="68.58" y1="-48.26" x2="66.04" y2="-48.26" width="0.1524" layer="91"/>
+<label x="66.04" y="-48.26" size="1.27" layer="95" rot="R180" xref="yes"/>
+</segment>
+</net>
+<net name="+3V3" class="0">
+<segment>
+<pinref part="U$3" gate="MSP432" pin="31"/>
+<wire x1="93.98" y1="50.8" x2="86.36" y2="50.8" width="0.1524" layer="91"/>
+<pinref part="+3V1" gate="G$1" pin="+3V3"/>
+</segment>
+<segment>
+<pinref part="U$2" gate="G$1" pin="3V3"/>
+<pinref part="+3V2" gate="G$1" pin="+3V3"/>
+</segment>
+<segment>
+<pinref part="U$1" gate="G$1" pin="VDD"/>
+<pinref part="+3V3" gate="G$1" pin="+3V3"/>
+</segment>
+<segment>
+<pinref part="U$4" gate="G$1" pin="VBATT"/>
+<wire x1="132.08" y1="48.26" x2="132.08" y2="45.72" width="0.1524" layer="91"/>
+<pinref part="+3V4" gate="G$1" pin="+3V3"/>
+</segment>
+<segment>
+<pinref part="U$5" gate="G$1" pin="3V3"/>
+<pinref part="+3V5" gate="G$1" pin="+3V3"/>
+</segment>
+</net>
+<net name="CD1" class="0">
+<segment>
+<pinref part="U$1" gate="G$1" pin="CARD_DETECT"/>
+<wire x1="81.28" y1="111.76" x2="78.74" y2="111.76" width="0.1524" layer="91"/>
+<label x="78.74" y="111.76" size="1.27" layer="95" rot="R180" xref="yes"/>
+</segment>
+<segment>
+<pinref part="U$3" gate="MSP432" pin="48"/>
+<wire x1="33.02" y1="-2.54" x2="33.02" y2="5.08" width="0.1524" layer="91"/>
+<label x="33.02" y="5.08" size="1.27" layer="95" rot="R90" xref="yes"/>
+</segment>
+</net>
+<net name="N$3" class="0">
+<segment>
+<pinref part="U$1" gate="G$1" pin="CARD_DETECT1"/>
+<wire x1="81.28" y1="109.22" x2="78.74" y2="109.22" width="0.1524" layer="91"/>
+</segment>
+</net>
+<net name="N$1" class="0">
+<segment>
+<pinref part="U$4" gate="G$1" pin="ANTENNA"/>
+<wire x1="154.94" y1="30.48" x2="175.26" y2="30.48" width="0.1524" layer="91"/>
+<pinref part="U$6" gate="G$1" pin="RF-IN"/>
+</segment>
+</net>
+<net name="N$6" class="0">
+<segment>
+<pinref part="U$6" gate="G$1" pin="RF-OUT"/>
+<pinref part="X1" gate="G$1" pin="ANT"/>
+<wire x1="215.9" y1="27.94" x2="198.12" y2="27.94" width="0.1524" layer="91"/>
+</segment>
+</net>
+<net name="VCC" class="0">
+<segment>
+<pinref part="BATTERY" gate="G$1" pin="2"/>
+<wire x1="-35.56" y1="45.72" x2="-25.4" y2="45.72" width="0.1524" layer="91"/>
+<pinref part="P+1" gate="VCC" pin="VCC"/>
+</segment>
+</net>
+<net name="VSS" class="0">
+<segment>
+<pinref part="BATTERY" gate="G$1" pin="1"/>
+<wire x1="-35.56" y1="43.18" x2="-25.4" y2="43.18" width="0.1524" layer="91"/>
+<pinref part="VSS1" gate="G$1" pin="VSS"/>
 </segment>
 </net>
@@
 </drawing>
 <compatibility>
+<note version="6.3" minversion="6.2.2" severity="warning">
+Since Version 6.2.2 text objects can contain more than one line,
+which will not be processed correctly with this version.
+</note>
 <note version="8.2" severity="warning">
 Since Version 8.2, EAGLE supports online libraries. The ids

Commit message: PDR schematic and board
Parts:
- removed U$5: TEENSY_3.5/3.6_BASIC, Teensy356:TEENSY_3.5/3.6_BASIC
- added SJ1, SJ2: (no value), jumper:SJ2WW
- added TEENSY: (no value), pinhead:PINHD-1X4
- added U1: V_REG_NCP50X, SparkFun-IC-Power:V_REG_NCP50X
Connections:
- new net N$7: SJ1.1, U1.IN
- new net N$8: SJ2.3, U1.OUT
- net +3V3: now also SJ2.2, TEENSY.4; no longer U$5.3V3
- net GND: now also TEENSY.1; no longer U$5.GND
- net TEENSY_RX: now also TEENSY.2; no longer U$5.0/RX
- net TEENSY_TX: now also TEENSY.3; no longer U$5.1/TX
- net VCC: now also SJ1.2
Other:
- moved on the sheet: BATTERY, C1, C2, C3, R1, R2, R3, U$2, X1

Commit message: Final board and schematic
Parts:
- added SD_BREAKOUT: (no value), pinhead:PINHD-1X7
Connections:
- removed net N$3: U$1.CARD_DETECT1
- net +3V3: now also SD_BREAKOUT.6
- net CD1: now also SD_BREAKOUT.1
- net GND: now also SD_BREAKOUT.7
- net SD_CLK: now also SD_BREAKOUT.4
- net SD_CS_SPI: now also SD_BREAKOUT.5
- net SD_MISO: now also SD_BREAKOUT.2
- net SD_MOSI: now also SD_BREAKOUT.3
Changed lines of the file:
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@@
 <part name="+3V6" library="supply1" library_urn="urn:adsk.eagle:library:371" deviceset="+3V3" device=""/>
 <part name="TEENSY" library="pinhead" library_urn="urn:adsk.eagle:library:325" deviceset="PINHD-1X4" device="" package3d_urn="urn:adsk.eagle:package:22407/2"/>
+<part name="SD_BREAKOUT" library="pinhead" library_urn="urn:adsk.eagle:library:325" deviceset="PINHD-1X7" device="" package3d_urn="urn:adsk.eagle:package:22477/2"/>
+<part name="+3V7" library="supply1" library_urn="urn:adsk.eagle:library:371" deviceset="+3V3" device=""/>
+<part name="GND14" library="supply1" library_urn="urn:adsk.eagle:library:371" deviceset="GND" device=""/>
 </parts>
 <sheets>
@@
 <attribute name="VALUE" x="21.59" y="91.44" size="1.778" layer="96"/>
 </instance>
+<instance part="SD_BREAKOUT" gate="A" x="104.14" y="91.44" smashed="yes">
+<attribute name="NAME" x="97.79" y="102.235" size="1.778" layer="95"/>
+<attribute name="VALUE" x="97.79" y="78.74" size="1.778" layer="96"/>
+</instance>
+<instance part="+3V7" gate="G$1" x="96.52" y="86.36" smashed="yes" rot="R90">
+<attribute name="VALUE" x="101.6" y="83.82" size="1.778" layer="96" rot="R180"/>
+</instance>
+<instance part="GND14" gate="1" x="96.52" y="83.82" smashed="yes" rot="R270">
+<attribute name="VALUE" x="93.98" y="86.36" size="1.778" layer="96" rot="R270"/>
+</instance>
 </instances>
 <busses>
@@
 <label x="38.1" y="2.54" size="1.27" layer="95" rot="R90" xref="yes"/>
 </segment>
+<segment>
+<pinref part="SD_BREAKOUT" gate="A" pin="5"/>
+<wire x1="101.6" y1="88.9" x2="99.06" y2="88.9" width="0.1524" layer="91"/>
+<label x="96.52" y="88.9" size="1.27" layer="95" rot="R180" xref="yes"/>
+</segment>
 </net>
 <net name="SD_CLK" class="0">
@@
 <label x="38.1" y="-15.24" size="1.27" layer="95" rot="R270" xref="yes"/>
 </segment>
+<segment>
+<pinref part="SD_BREAKOUT" gate="A" pin="4"/>
+<wire x1="101.6" y1="91.44" x2="99.06" y2="91.44" width="0.1524" layer="91"/>
+<label x="96.52" y="91.44" size="1.27" layer="95" rot="R180" xref="yes"/>
+</segment>
 </net>
 <net name="SD_MISO" class="0">
@@
 <label x="35.56" y="2.54" size="1.27" layer="95" rot="R90" xref="yes"/>
 </segment>
+<segment>
+<pinref part="SD_BREAKOUT" gate="A" pin="2"/>
+<wire x1="101.6" y1="96.52" x2="99.06" y2="96.52" width="0.1524" layer="91"/>
+<label x="96.52" y="96.52" size="1.27" layer="95" rot="R180" xref="yes"/>
+</segment>
 </net>
 <net name="SD_MOSI" class="0">
@@
 <wire x1="35.56" y1="-10.16" x2="35.56" y2="-15.24" width="0.1524" layer="91"/>
 <label x="35.56" y="-15.24" size="1.27" layer="95" rot="R270" xref="yes"/>
+</segment>
+<segment>
+<pinref part="SD_BREAKOUT" gate="A" pin="3"/>
+<wire x1="101.6" y1="93.98" x2="99.06" y2="93.98" width="0.1524" layer="91"/>
+<label x="96.52" y="93.98" size="1.27" layer="95" rot="R180" xref="yes"/>
 </segment>
 </net>
@@
 <wire x1="7.62" y1="104.14" x2="25.4" y2="104.14" width="0.1524" layer="91"/>
 </segment>
+<segment>
+<pinref part="SD_BREAKOUT" gate="A" pin="7"/>
+<wire x1="101.6" y1="83.82" x2="99.06" y2="83.82" width="0.1524" layer="91"/>
+<pinref part="GND14" gate="1" pin="GND"/>
+</segment>
 </net>
 <net name="N$2" class="0">
@@
 <wire x1="7.62" y1="96.52" x2="25.4" y2="96.52" width="0.1524" layer="91"/>
 </segment>
+<segment>
+<pinref part="SD_BREAKOUT" gate="A" pin="6"/>
+<wire x1="101.6" y1="86.36" x2="99.06" y2="86.36" width="0.1524" layer="91"/>
+<pinref part="+3V7" gate="G$1" pin="+3V3"/>
+</segment>
 </net>
 <net name="CD1" class="0">
@@
 <label x="33.02" y="5.08" size="1.27" layer="95" rot="R90" xref="yes"/>
 </segment>
-</net>
-<net name="N$3" class="0">
-<segment>
-<pinref part="U$1" gate="G$1" pin="CARD_DETECT1"/>
-<wire x1="53.34" y1="111.76" x2="50.8" y2="111.76" width="0.1524" layer="91"/>
-</segment>
-</net>
+<segment>
+<pinref part="SD_BREAKOUT" gate="A" pin="1"/>
+<wire x1="101.6" y1="99.06" x2="99.06" y2="99.06" width="0.1524" layer="91"/>
+<label x="96.52" y="99.06" size="1.27" layer="95" rot="R180" xref="yes"/>
+</segment>
+</net>
