File: PCB/ECEN 2440 Final Project/Radio Board.sch (EAGLE design)
At the start: 20 parts

Commit message: final (i hope) radio board
Parts:
- removed 3V3POWER: (no value), pinhead:PINHD-1X2
- removed LM317: LM317, Custom Library:LM317
- added 4VPWR: (no value), pinhead:PINHD-1X2
- added C4: 500n, rcl:C-USC0805
- added CIN1, CIN2: (no value), rcl:CPOL-USA
- added L1: (no value), rcl:L-USL3225M
- added R6: 0R, rcl:R-US_R0805
- added R8, R9: (no value), rcl:R-US_R0805
- added U$1: BD00COAW, Custom Library:BD00COAW
- R4: value 220R -> 43k
- R5: value 470R -> 10k
Connections:
- removed net +3V3: 3V3POWER.1, COUT.+, LM317.P$3, R4.2, R5.1, U$4.VBATT
- new net ADJ: R4.2, R5.1, U$1.ADJ
- new net GNDA: R6.1, U$6.GND1, X1.GND1, X1.GND2, X1.GND3, X1.GND4
- new net N$9: CIN1.+, R8.2
- new net V+: 4VPWR.1, C4.1, L1.2, R8.1, R9.1, U$4.VBATT
- new net VO: COUT.+, L1.1, R4.1, U$1.VO
- net GND: now also 4VPWR.2, C4.2, CIN1.-, CIN2.-, R6.2, U$1.GND; no longer 3V3POWER.2, U$6.GND1, X1.GND1, X1.GND2, X1.GND3, X1.GND4
- net N$8: now also CIN2.+, R9.2; no longer LM317.P$1, R4.1
- net VCC: now also U$1.CTL, U$1.VCC; no longer LM317.P$2
Other:
- note added: "VCC = battery input voltage V+ = +4Vout from vreg GND= common GND GNDA = RF ground"
- note removed: "LM317"
- moved on the sheet: BATT, CIN, COUT, R4, R5

Commit message: final board maybe??
Parts:
- U$1: value BD00COAW -> BDXXC0A-CBD00C0AWHFP-CTR; device Custom Library:BD00COAW -> Custom Library:BDXXC0A-CBD00C0AWHFP-CTR
Changed lines of the file:
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@@
 </class>
 <class number="2" name="pwr" width="0.889" drill="0.381">
-<clearance class="2" value="0.254"/>
+<clearance class="2" value="0.381"/>
+</class>
+<class number="3" name="gnd" width="0.508" drill="0">
+<clearance class="3" value="0.381"/>
+</class>
+<class number="4" name="rfgnd" width="0" drill="0">
+<clearance class="3" value="0.381"/>
 </class>
 </classes>
@@
 <part name="P+3" library="supply1" library_urn="urn:adsk.eagle:library:371" deviceset="VCC" device=""/>
 <part name="P+1" library="supply1" library_urn="urn:adsk.eagle:library:371" deviceset="V+" device=""/>
-<part name="U$1" library="Custom Library" deviceset="BD00COAW" device=""/>
+<part name="U$1" library="Custom Library" deviceset="BDXXC0A-C" device="BD00C0AWHFP-CTR"/>
 <part name="L1" library="rcl" library_urn="urn:adsk.eagle:library:334" deviceset="L-US" device="L3225M" package3d_urn="urn:adsk.eagle:package:23477/2"/>
 <part name="R8" library="rcl" library_urn="urn:adsk.eagle:library:334" deviceset="R-US_" device="R0805" package3d_urn="urn:adsk.eagle:package:23553/2"/>
@@
 </segment>
 </net>
-<net name="GND" class="0">
+<net name="GND" class="3">
 <segment>
 <pinref part="U$4" gate="G$1" pin="GND2"/>
@@
 </segment>
 </net>
-<net name="GNDA" class="0">
+<net name="GNDA" class="4">
 <segment>
 <pinref part="X1" gate="G$1" pin="GND3"/>

Commit message: naming
Parts:
- C1, C2, C3: value 500n -> (none)
- R1, R2, R3: value 100R -> 0R
- renumbered CIN1 to C5, CIN2 to C6
Changed lines of the file:
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@@
 <part name="U$4" library="Custom Library" deviceset="RADIO" device=""/>
 <part name="GND3" library="supply1" library_urn="urn:adsk.eagle:library:371" deviceset="GND" device=""/>
-<part name="R1" library="rcl" library_urn="urn:adsk.eagle:library:334" deviceset="R-US_" device="R0805" package3d_urn="urn:adsk.eagle:package:23553/2" value="100R"/>
-<part name="R2" library="rcl" library_urn="urn:adsk.eagle:library:334" deviceset="R-US_" device="R0805" package3d_urn="urn:adsk.eagle:package:23553/2" value="100R"/>
-<part name="R3" library="rcl" library_urn="urn:adsk.eagle:library:334" deviceset="R-US_" device="R0805" package3d_urn="urn:adsk.eagle:package:23553/2" value="100R"/>
-<part name="C1" library="rcl" library_urn="urn:adsk.eagle:library:334" deviceset="C-US" device="C0805" package3d_urn="urn:adsk.eagle:package:23617/2" value="500n"/>
-<part name="C2" library="rcl" library_urn="urn:adsk.eagle:library:334" deviceset="C-US" device="C0805" package3d_urn="urn:adsk.eagle:package:23617/2" value="500n"/>
-<part name="C3" library="rcl" library_urn="urn:adsk.eagle:library:334" deviceset="C-US" device="C0805" package3d_urn="urn:adsk.eagle:package:23617/2" value="500n"/>
+<part name="R1" library="rcl" library_urn="urn:adsk.eagle:library:334" deviceset="R-US_" device="R0805" package3d_urn="urn:adsk.eagle:package:23553/2" value="0R"/>
+<part name="R2" library="rcl" library_urn="urn:adsk.eagle:library:334" deviceset="R-US_" device="R0805" package3d_urn="urn:adsk.eagle:package:23553/2" value="0R"/>
+<part name="R3" library="rcl" library_urn="urn:adsk.eagle:library:334" deviceset="R-US_" device="R0805" package3d_urn="urn:adsk.eagle:package:23553/2" value="0R"/>
+<part name="C1" library="rcl" library_urn="urn:adsk.eagle:library:334" deviceset="C-US" device="C0805" package3d_urn="urn:adsk.eagle:package:23617/2"/>
+<part name="C2" library="rcl" library_urn="urn:adsk.eagle:library:334" deviceset="C-US" device="C0805" package3d_urn="urn:adsk.eagle:package:23617/2"/>
+<part name="C3" library="rcl" library_urn="urn:adsk.eagle:library:334" deviceset="C-US" device="C0805" package3d_urn="urn:adsk.eagle:package:23617/2"/>
 <part name="GND6" library="supply1" library_urn="urn:adsk.eagle:library:371" deviceset="GND" device=""/>
 <part name="GND7" library="supply1" library_urn="urn:adsk.eagle:library:371" deviceset="GND" device=""/>
@@
 <part name="R9" library="rcl" library_urn="urn:adsk.eagle:library:334" deviceset="R-US_" device="R0805" package3d_urn="urn:adsk.eagle:package:23553/2"/>
 <part name="GND2" library="supply1" library_urn="urn:adsk.eagle:library:371" deviceset="GND" device=""/>
-<part name="CIN1" library="rcl" library_urn="urn:adsk.eagle:library:334" deviceset="CPOL-US" device="A" package3d_urn="urn:adsk.eagle:package:23418/2"/>
-<part name="CIN2" library="rcl" library_urn="urn:adsk.eagle:library:334" deviceset="CPOL-US" device="A" package3d_urn="urn:adsk.eagle:package:23418/2"/>
+<part name="C5" library="rcl" library_urn="urn:adsk.eagle:library:334" deviceset="CPOL-US" device="A" package3d_urn="urn:adsk.eagle:package:23418/2"/>
+<part name="C6" library="rcl" library_urn="urn:adsk.eagle:library:334" deviceset="CPOL-US" device="A" package3d_urn="urn:adsk.eagle:package:23418/2"/>
 <part name="C4" library="rcl" library_urn="urn:adsk.eagle:library:334" deviceset="C-US" device="C0805" package3d_urn="urn:adsk.eagle:package:23617/2" value="500n"/>
 </parts>
@@
 <attribute name="VALUE" x="15.24" y="55.88" size="1.778" layer="96"/>
 </instance>
-<instance part="CIN1" gate="G$1" x="104.14" y="96.52" smashed="yes">
+<instance part="C5" gate="G$1" x="104.14" y="96.52" smashed="yes">
 <attribute name="NAME" x="105.156" y="97.155" size="1.778" layer="95"/>
 <attribute name="VALUE" x="105.156" y="92.329" size="1.778" layer="96"/>
 </instance>
-<instance part="CIN2" gate="G$1" x="116.84" y="96.52" smashed="yes">
+<instance part="C6" gate="G$1" x="116.84" y="96.52" smashed="yes">
 <attribute name="NAME" x="117.856" y="97.155" size="1.778" layer="95"/>
 <attribute name="VALUE" x="117.856" y="92.329" size="1.778" layer="96"/>
@@
 <wire x1="116.84" y1="91.44" x2="116.84" y2="86.36" width="0.1524" layer="91"/>
 <junction x="116.84" y="86.36"/>
-<pinref part="CIN2" gate="G$1" pin="-"/>
-<pinref part="CIN1" gate="G$1" pin="-"/>
+<pinref part="C6" gate="G$1" pin="-"/>
+<pinref part="C5" gate="G$1" pin="-"/>
 </segment>
 <segment>
@@
 <pinref part="R9" gate="G$1" pin="2"/>
 <wire x1="116.84" y1="101.6" x2="116.84" y2="99.06" width="0.1524" layer="91"/>
-<pinref part="CIN2" gate="G$1" pin="+"/>
+<pinref part="C6" gate="G$1" pin="+"/>
 </segment>
 </net>
@@
 <pinref part="R8" gate="G$1" pin="2"/>
 <wire x1="104.14" y1="101.6" x2="104.14" y2="99.06" width="0.1524" layer="91"/>
-<pinref part="CIN1" gate="G$1" pin="+"/>
-</segment>
-</net>
+<pinref part="C5" gate="G$1" pin="+"/>
+</segment>
+</net>

Commit message: really important commit
Parts:
- added U$2: WOBBUFFET, Custom Library:WOBBUFFET
Changed lines of the file:
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@@
 <part name="C6" library="rcl" library_urn="urn:adsk.eagle:library:334" deviceset="CPOL-US" device="A" package3d_urn="urn:adsk.eagle:package:23418/2"/>
 <part name="C4" library="rcl" library_urn="urn:adsk.eagle:library:334" deviceset="C-US" device="C0805" package3d_urn="urn:adsk.eagle:package:23617/2" value="500n"/>
+<part name="U$2" library="Custom Library" deviceset="WOBBUFFET" device=""/>
 </parts>
 <sheets>
@@
 <attribute name="NAME" x="18.796" y="69.215" size="1.778" layer="95"/>
 </instance>
+<instance part="U$2" gate="G$1" x="109.22" y="76.2" smashed="yes"/>
 </instances>
 <busses>
